File: Schematics/moonclock/moonclock.kicad_pcb (KiCad board)
At the start: 2 copper layers, 50 x 80 mm, 29 parts, among them J1 Conn_01x05, J2 Screw_Terminal_01x04, J3 Screw_Terminal_01x03, J4 Conn_01x04, J5 Conn_01x04, U1 RP2040-Zero, U2 MCP4922-ESL, U3 MAX6071AAUT21+T, U4 MCP6002-xSN

Commit message: Minor PCB updates
Other:
- board text added: "+3.3V"
Changed lines of the file:
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@@
 		(layer "F.CrtYd")
 	)
-	(gr_text "+5V"
+	(gr_text "+3.3V"
 		(at 160 77.65 0)
 		(layer "F.SilkS")

Commit message: Start on rev 2 design
Parts:
- added BT1: Battery_Cell, bs7:BAT_BS-7, F.Cu at (94.1, 97.0)
- added U5: MCP7940N-xSN, Package_SO:SOIC-8_3.9x4.9mm_P1.27mm, F.Cu at (67.7, 115.2)
Connections:
- J4 pad 1: GND -> I2C1_SCL
- J4 pad 2: +3.3V -> I2C1_SDA
- J4 pad 3: I2C1_SDA -> +3.3V
- J4 pad 4: I2C1_SCL -> GND
