File: Schematics/moonclock/moonclock.kicad_pcb (KiCad board)
At the start: 2 copper layers, 50 x 80 mm, 32 parts, among them J1 Conn_01x06, J2 Conn_01x04, J3 Screw_Terminal_01x04, J4 Screw_Terminal_01x04, J5 Screw_Terminal_01x04, J6 Conn_01x04, J7 Conn_01x05, U1 RP2040-Zero, U2 MCP6002-xSN, U3 MCP47FVB22-E/ST, U4 MCP7940N-xSN, Y1 ECS-.327-6-17X-C-TR

Commit message: Schematic cosmetic improvements and PDF plot
Connections:
- net DISP_CS renamed ~{DISP_CS}
